File: AscPcb.kicad_pcb (KiCad board)
At the start: 2 copper layers, 82.7 x 79.3 mm, 88 parts, among them J1 12402012E212A, J10 Conn_01x02_Pin, J15 Conn_01x02_Pin, J16 Conn_01x02_Pin, J17 Conn_01x02_Pin, J2 B2B-PH-K-S(LF)(SN), J3 Screw_Terminal_01x02, J4 Screw_Terminal_01x02, J5 Conn_01x15_Pin, J6 Conn_01x06_Pin, J7 Conn_01x02_Pin, J8 Conn_01x02_Pin, Q1 Q_NMOS_DGS, Q2 BC817, Q3 BC817, SW1 TL3305AF260QG, SW2 TL3305AF260QG, U1 BQ24040DSQR, U2 TLV75801PDRVR, U3 AP62300TWU, U4 LTC3625EDE_PBF, U5 ESP32-C3-WROOM-02-N4, U6 CP2102N-A02-GQFN24R, U7 BMI270, U8 74LVC1G07

Commit message: routing done not gnd
Connections:
- J5 pad 10: IO7 -> IO4
- J5 pad 11: IO10 -> IO3
- J5 pad 12: IO18 -> IO1
- J5 pad 13: IO19 -> IO0
- J5 pad 14: ESP_TXD -> ESP_RXD
- J5 pad 15: ESP_RXD -> ESP_TXD
- J5 pad 4: IO0 -> IO19
- J5 pad 5: IO1 -> IO18
- J5 pad 6: IO3 -> IO10
- J5 pad 7: IO4 -> IO7
- J5 pad 8: IO5 -> IO6
- J5 pad 9: IO6 -> IO5
Routing:
- net +3V3: track 16.4 -> 166.4 mm, vias 0 -> 6
- net IO3: track 1.66 -> 106.3 mm, vias 0 -> 8
- net EN: track 0.00 -> 77.9 mm, vias 0 -> 4
- net IO1: track 1.55 -> 67.7 mm
- net IO0: track 3.96 -> 69.4 mm
- net IO6: track 0.00 -> 60.7 mm, vias 0 -> 4
- net IO9: track 0.00 -> 58.1 mm, vias 0 -> 2
- net IO7: track 0.00 -> 45.5 mm, vias 0 -> 7
- net IO5: track 0.00 -> 45.2 mm, vias 0 -> 3
- net IO4: track 0.00 -> 44.0 mm, vias 0 -> 4
- net IO10: track 0.00 -> 29.5 mm, vias 0 -> 1
- net POWER: track 38.0 -> 66.9 mm
- net IO19: track 10.9 -> 39.2 mm, vias 0 -> 2
- net IO18: track 10.7 -> 34.2 mm, vias 0 -> 2
- net ESP_RXD: track 49.2 -> 66.0 mm, vias 0 -> 1
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